File: freeduino_hs.brd (EAGLE design)
At the start: 68.6 x 53.3 mm, 46 parts, among them J1 DC-005, Q1 16 MHz, Q2 12 MHz, T1 FDN340P, U1 CH340G, U2 LM393D, U3 ATMEGA328P-PU, U4 REG1117, U5 REG1117, X1 MINI-USB-32005-201

Commit message: Some optimizations
Parts:
- moved R9 6.31 mm to (52.3, 23.7), turned to 270 degrees
- moved C3 2.81 mm to (56.8, 27.6)
Routing:
- net N$4: track 4.57 -> 7.61 mm
- net GND: track 17.0 -> 19.7 mm, vias 31 -> 27
- net AD4/SDA: track 92.2 -> 89.7 mm
- net DTR: track 40.4 -> 38.4 mm
- net IO2: track 36.7 -> 34.8 mm
- net N$1: track 3.62 -> 5.18 mm
- net +5V: track 179.9 -> 181.3 mm, vias 4 -> 6
- net IO7: track 41.8 -> 40.7 mm
- net USBVCC: track 31.7 -> 30.6 mm
- net SCK: track 113.4 -> 112.3 mm
- net RESET: track 136.7 -> 135.7 mm
- net IO0: track 84.6 -> 83.9 mm
- net IO3: track 34.8 -> 35.4 mm
- net AD5/SCL: track 94.0 -> 93.4 mm
- added copper zone on layer 16, net N$92
- removed copper zone on layer 1, net N$92
Other:
- board text removed: "L"
- board text removed: "PC1"
- board text removed: "PC2"
